File: fibonacci_clock_pcb/fibonacci_clock_pcb.kicad_pcb (KiCad board)
At the start: 2 copper layers, 105 x 90 mm, 12 parts, among them J1 Top 16, J2 Bottom 16, J3 Jack-DC, U1 Cathode, U2 Red, U3 Green, U4 Blue, U5 WeMos_D1_mini

Commit message: Added the new images and the production images
Parts:
- added G***: LOGO, Assets:logo, F.Cu at (39.0, 100.0)
- moved J3 3.36 mm to (78.0, 22.3), turned to 180 degrees
Connections:
- J3 pad 3: GND -> (no net)
- U5 pad 13: CRGB_DataIN -> unconnected-(U5-SDA/D2-Pad13)
- U5 pad 14: CRGB_ClockPin -> unconnected-(U5-SCL/D1-Pad14)
- U5 pad 3: CRGB_LatchPin -> unconnected-(U5-D0-Pad3)
- U5 pad 4: unconnected-(U5-SCK/D5-Pad4) -> CRGB_ClockPin
- U5 pad 5: unconnected-(U5-MISO/D6-Pad5) -> CRGB_DataIN
- U5 pad 7: unconnected-(U5-CS/D8-Pad7) -> CRGB_LatchPin
Routing:
- net CRGB_ClockPin: track 262.3 -> 280.7 mm
- net CRGB_DataIN: track 102.6 -> 120.6 mm
- net CRGB_LatchPin: track 285.5 -> 280.6 mm
- net VCC: track 467.8 -> 465.2 mm
- net GND: track 475.8 -> 475.4 mm, vias 0 -> 7
Other:
- board text added: "26/10/2024"
- board text added: "V1.0"
