File: fibonacci_clock_pcb/fibonacci_clock_pcb.kicad_sch (KiCad schematic)
At the start: 12 parts, among them J1 Top 16, J2 Bottom 16, J3 Jack-DC, U1 Cathode, U2 Red, U3 Green, U4 Blue, U5 WeMos_D1_mini

Commit message: Added the new images and the production images
Connections:
- net CRGB_ClockPin: now also U5.4 (SCK/D5); no longer U5.14 (SCL/D1)
- net CRGB_DataIN: now also U5.5 (MISO/D6); no longer U5.13 (SDA/D2)
- net CRGB_LatchPin: now also U5.7 (CS/D8); no longer U5.3 (D0)
